File: mercury-1/mercury-1/mercury-1.kicad_sch (KiCad schematic)
At the start: 1 part, among them U1 XT60PW-F

Commit message: Started Power System
Parts:
- removed U1: XT60PW-F, logic_board:TH_2P-XT60PW-F, symbol logic_board:XT60PW-F_C428722
Other:
- note added: "= Logic Power"
- note added: "= Power Sequencing Control"
- note removed: "= Power"
- note removed: "= Power Sequencing"
- note removed: "Logic Rover Subsystem Requirements"

Commit message: breaking things just to fix them
Other:
- sheet Logic Power Subsystem renamed Power Subsystems
- sheet On-Board Sensors renamed Sensors and Serial Multiplexers
- sheet Rover Subsystems renamed Science Subsystem
- added sheet Arm Subsystem (untitled.kicad_sch)
- note added: "Rover Topology"
- note added: "Schematic Block Diagram"
- note removed: "Concept of Operations"
- note removed: "Ext. Power"
- note removed: "Power Input"
- note removed: "System Block Diagram"
