File: mercury-1/mercury-1/power.kicad_sch (KiCad schematic)
At the start: 0 parts

Commit message: Started Power System
Parts:
- added C1, C2, C3: 10uF, symbol Device:C
- added C23: 22n, EPS:C0402, symbol Device:C
- added C25: 2.2u, EPS:C0402, symbol Device:C
- added C26: 10p, EPS:C0402, symbol Device:C
- added C27, C28: 100n, EPS:C0402, symbol Device:C
- added C4: 220n, EPS:C0402, symbol Device:C
- added C52, C56: 47u, EPS:CAP-SMD_L7.3-W4.3-FD, symbol Device:C
- added L2: 6.1u, EPS:IND-SMD_FTKB1207-6R1NT, symbol Device:L
- added P1: Logic Kill Switch, Stuff:CONN-TH_2P-P5.00_WJ500V-5.08-2P, symbol logic_board:WJ500V-5.08-2P-14-00A
- added R1, R41, R59, R60, R61: 15k, EPS:R0402, symbol Device:R_US
- added R57: 1k, EPS:R0402, symbol Device:R_US
- added R62: 110k, EPS:R0402, symbol Device:R_US
- added R63: 47k, EPS:R0402, symbol Device:R_US
- added R64: 2k, EPS:R0402, symbol Device:R_US
- added R65: 240k, EPS:R0402, symbol Device:R_US
- added R66: 100k, EPS:R0402, symbol Device:R_US
- added TP1, TP10: TestPoint, TestPoint:TestPoint_Pad_1.0x1.0mm, symbol EPS:TestPoint
- added U1: XT60PW-F, logic_board:TH_2P-XT60PW-F, symbol logic_board:XT60PW-F_C428722
- added U2: TPS1HA08AQPWPRQ1, logic_board:HTSSOP-16_L5.0-W4.4-P0.65-LS6.4-BL-EP, symbol logic_board:TPS1HA08AQPWPRQ1
- added U3: LT8612EUDE#PBF, EPS:QFN-28_L6.0-W3.0-P0.50-BL-EP, symbol EPS:LT8612EUDE#PBF
Connections:
- new net: C23.1, R63.1, TP10.1, U2.6 (VOUT), U3.5 (VIN)
- new net: R63.2, R64.1, U3.4 (EN/UV)
- new net: C23.2, R59.2, R60.2, R61.2, U2.1 (GND)
- new net: R59.1, U2.16 (DIA_EN)
- new net: C26.2, R65.2, R66.1, U3.24 (FB)
- new net: C26.1, C52.1, C56.1, L2.2, R65.1, U3.22 (BIAS)
- new net: R1.1, U2.4 (EN)
- new net: P1.2, U1.3 (+)
- new net: R61.1, U2.14 (SEL1)
- new net: R60.1, U2.15 (SEL2)
- new net: C27.1, U3.20 (BST)
- new net: C27.2, L2.1, U3.15 (SW)
- new net: R57.2, U2.2 (SNS)
- new net: R41.2, U2.3 (LATCH)
- new net: R62.1, U3.3 (RT)
- new net: C28.1, U3.21 (INTVCC)
- new net: C25.1, U3.2 (TR/SS)
- new net +28V: C1.1, C2.1, C3.1, C4.1, P1.1, R1.2, TP1.1, U2.17 (VBB)
- new net GND: C1.2, C2.2, C25.2, C28.2, C3.2, C4.2, C52.2, C56.2, R41.1, R57.1, R62.2, R64.2, R66.2, U1.4 (-), U3.11 (GND), U3.25 (NC), U3.8 (PGND)
- new net GNDPWR: U1.1, U1.2
- no-connect marks 0 -> 5
Other:
- note added: "Raspberry Pi 4B Power Load Switch and Switching Regulator"

Commit message: breaking things just to fix them
Other:
- company: (none) -> BILLEE Rover
Changed lines of the file:
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@@
 	(generator_version "9.0")
 	(paper "A4")
+	(title_block
+		(company "BILLEE Rover")
+	)
 	(rectangle
 		(start 13.462 13.462)
@@
 		(margins 0.9525 0.9525 0.9525 0.9525)
 		(stroke
+			(width 0)
+			(type solid)
+		)
+		(fill
+			(type none)
+		)
+		(effects
+			(font
+				(size 1.27 1.27)
+			)
+			(justify left top)
+		)
+	)
+	(text_box "This power subsystem needs to be able to power sequence the following from their respective batteries.\nArm/Science can share the same battery pack -> Must use a relay triggered by the OBC. GPIO/Serial breakout for Arm. Repurpose for Science.\nComms/RF can use a load switch + switching regulator and draw power from the Logic board depending on the power requirements.\nEthernet Switch can use a load switch + switching regulator and draw power from the Logic Board depending on the power requirements.\nJetson can use load switch + switching regulator and draw power from teh Logic Board depending on the power draw."
+		(exclude_from_sim no)
+		(at 204.216 139.192 0)
+		(size 79.756 25.146)
+		(margins 0.9525 0.9525 0.9525 0.9525)
+		(stroke
