File: mercury-1/mercury-1/sensors.kicad_sch (KiCad schematic)
At the start: 0 parts

Commit message: breaking things just to fix them
Other:
- company: (none) -> BILLEE Rover
Changed lines of the file:
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@@
 	(generator_version "9.0")
 	(paper "A4")
+	(title_block
+		(company "BILLEE Rover")
+	)
 )
