File: mercury-1/mercury-1.kicad_sch (KiCad schematic)
At the start: 22 parts, among them J1 +22.2V Logic Battery Array, J2 +14.4V Drivetrain Battery Arr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, J3 +14.4V Drivetrain Battery Arr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, K1 100A Relay / 12VDC Coil, K2 100A Relay / 12VDC Coil, K3 100A Relay / 12VDC Coil, K4 100A Relay / 12VDC Coil, K5 100A Relay / 12VDC Coil, K6 100A Relay / 12VDC Coil, K7 100A Relay / 12VDC Coil, K8 100A Relay / 12VDC Coil, SW1 KSW, U1 UVLO Relay, U2 Buck Converter, U3 Buck Converter, U4 UVLO Relay, U5 Logic Relay, U6 Logic Relay, U7 UVLO Relay

Commit message: stuff
Parts:
- added BT1, BT2, BT3, BT4, BT5, BT6: Battery, symbol Device:Battery
- added TC1, TC2, TC3, TC4, TC5, TC6: K-Type, symbol Device:Thermocouple
- added U10, U11, U12, U13, U14, U9: MAX6675 Breakout, symbol logic_board:MAX6675_Breakout
- added U8: RASPBERRY_PI_4B_4GB, RASPBERRY_PI_4B_4GB:MODULE_RASPBERRY_PI_4B_4GB, symbol logic_board:RASPBERRY_PI_4B_4GB
Connections:
- net +14.4V: now also BT3.1 (+), BT4.1 (+)
- net +22.2V Arm/Science: now also BT5.1 (+), BT6.1 (+)
- net +22.2V Logic: now also BT1.1 (+), BT2.1 (+)
- net GND: now also BT1.2 (-), BT2.2 (-), BT3.2 (-), BT4.2 (-), BT5.2 (-), BT6.2 (-), U10.1 (GND), U11.1 (GND), U12.1 (GND), U13.1 (GND), U14.1 (GND), U8.14 (GND), U8.20 (GND), U8.25 (GND), U8.30 (GND), U8.34 (GND), U8.39 (GND), U8.6 (GND), U8.9 (GND), U9.1 (GND)
- net Arm/Science_VCC renamed Arm/Science_VCC
- net PI_GPIO1 renamed PI_GPIO5
- net PI_GPIO5: now also U8.29 (GPIO5)
- net PI_GPIO2 renamed PI_GPIO6
- net PI_GPIO6: now also U8.31 (GPIO6)
- new net: TC3.1 (+), U10.5 (+)
- new net: TC3.2 (-), U10.6 (-)
- new net: U11.3 (SCK), U14.3 (SCK)
- new net: U10.5 (+), U11.5 (+), U12.5 (+), U13.5 (+), U14.5 (+), U9.5 (+)
- new net: TC5.1 (+), U11.5 (+)
- new net: TC5.2 (-), U11.6 (-)
- new net: U12.3 (SCK), U9.3 (SCK)
- new net: TC2.1 (+), U12.5 (+)
- new net: TC2.2 (-), U12.6 (-)
- new net: TC6.1 (+), U14.5 (+)
- new net: TC6.2 (-), U14.6 (-)
- new net: TC4.1 (+), U13.5 (+)
- new net: TC4.2 (-), U13.6 (-)
- new net: U10.3 (SCK), U13.3 (SCK)
- new net: TC1.1 (+), U9.5 (+)
- new net: TC1.2 (-), U9.6 (-)
- new net 3V3: U8.1 (3V3), U8.17 (3V3)
- new net 5V: U10.2 (VCC), U11.2 (VCC), U12.2 (VCC), U13.2 (VCC), U14.2 (VCC), U8.2 (5V), U8.4 (5V), U9.2 (VCC)
- new net PI_GPIO12: U8.32 (GPIO12), U9.4 (CS)
- new net PI_GPIO13: U12.4 (CS), U8.33 (GPIO13)
- new net PI_GPIO16: U10.4 (CS), U8.36 (GPIO16)
- new net PI_GPIO19: U13.4 (CS), U8.35 (GPIO19)
- new net PI_GPIO20: U11.4 (CS), U8.38 (GPIO20)
- new net PI_GPIO21: U14.4 (CS), U8.40 (GPIO21)
- new net SHIELD: U8.S1 (SHIELD), U8.S2 (SHIELD), U8.S3 (SHIELD), U8.S4 (SHIELD)
- no-connect marks 3 -> 25
Other:
- note added: "Battery Arrays"
- note added: "Drivetrain 14.4v"
- note added: "Logic +22.2v"
- note added: "RPI4B GPIO Pinout"
- note added: "To Jetson USB Port"
- note removed: "= Ethernet"
- note removed: "= Logic Power"
- note removed: "= Power Sequencing Control"
- note removed: "= Serial Protocols"
- note removed: "Signal Legend"
- moved on the sheet: CB1, CB2, CB3, J1, J2, J3, K1, K2, K3, K4, K5, K6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

Commit message: Added more stuff
Parts:
- removed K1, K2, K3, K4, K5, K6, K7, K8: 100A Relay / 12VDC Coil, Relay_THT:Relay_SPST-NO_Fujitsu_FTR-LYAA005x_FormA_Vertical, symbol Relay:Fujitsu_FTR-LYAA005x
- removed SW1: KSW, Button_Switch_SMD:Nidec_Copal_CAS-120A, symbol Switch:SW_Nidec_CAS-120A1
- added J4: Jetson, symbol logic_board:JetsonGPIO
- added K1, K2, K3, K4, K5, K6, K7, K8: 200A Relay 12V Coil, symbol logic_board:200A Relay 12V Coil
- added SW1: SW_SPDT_321, symbol logic_board:SW_SPDT_321
- BT1, BT2, BT5, BT6: value Battery -> +22.2v 10Ah
- BT3, BT4: value Battery -> +14.8v 10Ah
- CB1, CB2, CB3: symbol Device:CircuitBreaker_1P -> logic_board:CircuitBreaker_1P
Connections:
- net +20V_Jetson: now also J4.41 (Pin_41)
- net +22.2V Logic: now also U1.2 (OUT+), U1.4 (V+), U1.5 (NO), K1.A1; no longer U1.1 (IN+)
- net Drivetrain_VCC: now also K5.13
- net GND: now also U1.1 (OUT-), U1.3 (V-), U4.1 (OUT-), U4.3 (V-), U7.1 (OUT-), U7.3 (V-), K2.A2, K4.A2, K5.A2, K6.A2, K8.A2, SW1.2 (B); no longer U1.2 (IN-), U1.4 (OUT-), U4.2 (IN-), U4.4 (OUT-), U7.2 (IN-), U7.4 (OUT-)
- net GND_Jetson: now also J4.42 (Pin_42)
- net KSW_GND: now also K1.A2, K3.A2, K7.A2, SW1.3 (A)
- net at U6.4 (NO): now also K8.A1
- net at CB2.1: now also K3.14
- net PI_SCK: now reaches U11.3 (SCK), U14.3 (SCK)
- net PI_SCK: now also U10.3 (SCK), U12.3 (SCK), U13.3 (SCK), U8.23 (GPIO11/SPI_SCLK), U9.3 (SCK)
- net PI_MISO: now reaches U10.5 (+), U11.5 (+), U12.5 (+), U13.5 (+), U14.5 (+), U9.5 (+)
- net PI_MISO: now also U8.21 (GPIO9/SPI_MISO)
- net at U2.8 (In+), U3.8 (In+): now also K2.13
- net at CB1.1: now also K1.14
- net at U5.4 (NO): now also K5.A1
- net at CB3.1: now also K7.14
- net +14.4V renamed +14.8V
- net +14.8V: now also U4.2 (OUT+), U4.4 (V+), U4.5 (NO), K3.A1; no longer U4.1 (IN+)
- net +22.2V Arm/Science renamed +22.2V A/S
- net +22.2V A/S: now also U7.2 (OUT+), U7.4 (V+), U7.5 (NO), K7.A1, K8.13; no longer U7.1 (IN+)
- new net: K1.13, K2.14
- new net: K2.A1, U1.5 (NO)
- new net: K6.13, K8.14
- new net: K6.14, K7.13
- new net: K6.A1, U7.5 (NO)
- new net: K4.13, K5.14
- new net: K3.13, K4.14
- new net: K4.A1, U4.5 (NO)
- no-connect marks 25 -> 26
Other:
- note added: "Drivetrain +14.8v"
- note added: "Jetson"
- note added: "RPI4B"
- note added: "Thermocouple Sensor Array"
- note added: "To PI4B USB"
- note removed: "Drivetrain 14.4v"
- note removed: "RPI4B GPIO Pinout"
- moved on the sheet: TC1, TC2, TC3, TC4, TC5, TC6, U10, U11, U12, U13, U14, U2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

Commit message: Updated
Changed all axis instead of 2 and 3 on arm to yellowjackets. Frank and Justin now need to redesign. Added Drivetrain, and Arm Motors, Drivers, and found encoder solution.
Parts:
- added J5: POE Injector, symbol Connector:Screw_Terminal_01x03
- added J6: Network Switch, symbol Connector:Screw_Terminal_01x03
- added J7: P-20-90-PRO-121-B, symbol logic_board:P-17-80-PRO-51-B
- added J8: P-20-90-PRO-121-B, symbol logic_board:P-20-90-PRO-121-B
- added M1, M2, M3, M4: Yellowjacket 5203, symbol logic_board:Yellowjacket 5203
- added M10, M5, M6, M7, M8, M9: NEO_Brushless_Motor, symbol logic_board:NEO_Brushless_Motor
- added R1, R2, R3, R4, R5, R6: 2 (50W), symbol Device:R_US
- added U15, U16, U17: RoboClaw_2x7A, symbol logic_board:RoboClaw_2x7A
- added U18, U19, U20, U21, U22, U23: ODESC_V4.2, symbol logic_board:ODESC_V4.2
- J3: value +14.4V Drivetrain Battery Array -> +22.2V A/S Battery Array
Connections:
- net +12V_Comms: now also J5.3 (Pin_3), J6.3 (Pin_3)
- net +22.2V A/S: no longer K8.13
- net Drivetrain_VCC: now also U18.1 (VBAT+), U19.1 (VBAT+), U20.1 (VBAT+), U21.1 (VBAT+), U22.1 (VBAT+), U23.1 (VBAT+)
- net GND: now also J7.3 (CANH), J8.3 (CANH), U15.36 (M_GND), U16.36 (M_GND), U17.36 (M_GND), U18.2 (GND), U19.2 (GND), U20.2 (GND), U21.2 (GND), U22.2 (GND), U23.2 (GND)
- net GND_Comms: now also J5.2 (Pin_2), J6.2 (Pin_2)
- net GPIO8: now reaches J4.16 (Pin_16)
- net GPIO8: now also U15.3 (S1), U16.3 (S1), U17.3 (S1)
- net GPIO35: now reaches J4.18 (Pin_18)
- net GPIO35: now also U16.7 (S2)
- net Jetson_+5V: now reaches J4.2 (Pin_2)
- net Jetson_+5V: now also U15.1 (LB_IN+), U16.1 (LB_IN+), U17.1 (LB_IN+)
- net GPIO17: now reaches J4.22 (Pin_22)
- net GPIO17: now also U15.7 (S2), U17.7 (S2)
- net Jetson_GND: now reaches J4.6 (Pin_6)
- net Jetson_GND: now also U15.10 (S2_GND), U15.2 (LB_IN-), U16.10 (S2_GND), U16.2 (LB_IN-), U17.10 (S2_GND), U17.2 (LB_IN-)
- new net: M10.5 (ENC_C/Z), U23.10 (ENC_A_I)
- new net: M10.9 (ENC_5V), U23.11 (ENC_A_5V)
- new net: M10.4 (ENC_GND), U23.12 (ENC_A_GND)
- new net: M10.1 (PHASE_A), U23.3 (MOTOR_A)
- new net: M10.2 (PHASE_B), U23.4 (MOTOR_B)
- new net: M10.3 (PHASE_C), U23.5 (MOTOR_C)
- new net: R6.1, U23.6 (RES+)
- new net: R6.2, U23.7 (RES-)
- new net: M10.7 (ENC_A), U23.8 (ENC_A_A)
- new net: M10.6 (ENC_B), U23.9 (ENC_A_B)
- new net: M7.1 (PHASE_A), U20.3 (MOTOR_A)
- new net: M7.2 (PHASE_B), U20.4 (MOTOR_B)
- new net: M7.3 (PHASE_C), U20.5 (MOTOR_C)
- new net: M7.4 (ENC_GND), U20.12 (ENC_A_GND)
- new net: M7.5 (ENC_C/Z), U20.10 (ENC_A_I)
- new net: M7.6 (ENC_B), U20.9 (ENC_A_B)
- new net: M7.7 (ENC_A), U20.8 (ENC_A_A)
- new net: M7.9 (ENC_5V), U20.11 (ENC_A_5V)
- new net: M5.5 (ENC_C/Z), U18.10 (ENC_A_I)
- new net: M5.9 (ENC_5V), U18.11 (ENC_A_5V)
- new net: M5.4 (ENC_GND), U18.12 (ENC_A_GND)
- new net: M5.1 (PHASE_A), U18.3 (MOTOR_A)
- new net: M5.2 (PHASE_B), U18.4 (MOTOR_B)
- new net: M5.3 (PHASE_C), U18.5 (MOTOR_C)
- new net: R1.1, U18.6 (RES+)
- new net: R1.2, U18.7 (RES-)
- new net: M5.7 (ENC_A), U18.8 (ENC_A_A)
- new net: M5.6 (ENC_B), U18.9 (ENC_A_B)
- new net: R3.1, U20.6 (RES+)
- new net: R3.2, U20.7 (RES-)
- new net: M9.5 (ENC_C/Z), U22.10 (ENC_A_I)
- new net: M9.9 (ENC_5V), U22.11 (ENC_A_5V)
- new net: M9.4 (ENC_GND), U22.12 (ENC_A_GND)
- new net: M9.1 (PHASE_A), U22.3 (MOTOR_A)
- new net: M9.2 (PHASE_B), U22.4 (MOTOR_B)
- new net: M9.3 (PHASE_C), U22.5 (MOTOR_C)
- new net: R5.1, U22.6 (RES+)
- new net: R5.2, U22.7 (RES-)
- new net: M9.7 (ENC_A), U22.8 (ENC_A_A)
- new net: M9.6 (ENC_B), U22.9 (ENC_A_B)
- new net: M6.5 (ENC_C/Z), U19.10 (ENC_A_I)
- new net: M6.9 (ENC_5V), U19.11 (ENC_A_5V)
- new net: M6.4 (ENC_GND), U19.12 (ENC_A_GND)
- new net: M6.1 (PHASE_A), U19.3 (MOTOR_A)
- new net: M6.2 (PHASE_B), U19.4 (MOTOR_B)
- new net: M6.3 (PHASE_C), U19.5 (MOTOR_C)
- new net: R2.1, U19.6 (RES+)
- new net: R2.2, U19.7 (RES-)
- new net: M6.7 (ENC_A), U19.8 (ENC_A_A)
- new net: M6.6 (ENC_B), U19.9 (ENC_A_B)
- new net: M8.1 (PHASE_A), U21.3 (MOTOR_A)
- new net: M8.2 (PHASE_B), U21.4 (MOTOR_B)
- new net: M8.3 (PHASE_C), U21.5 (MOTOR_C)
- new net: M8.4 (ENC_GND), U21.12 (ENC_A_GND)
- new net: M8.5 (ENC_C/Z), U21.10 (ENC_A_I)
- new net: M8.6 (ENC_B), U21.9 (ENC_A_B)
- new net: M8.7 (ENC_A), U21.8 (ENC_A_A)
- new net: M8.9 (ENC_5V), U21.11 (ENC_A_5V)
- new net: R4.1, U21.6 (RES+)
- new net: R4.2, U21.7 (RES-)
- new net +22.2V_Arm/Science_OUT: J7.4 (CANL), J8.4 (CANL), K8.13, U15.36 (M_GND), U16.36 (M_GND), U17.36 (M_GND)
- new net Axis_1+: M1.1 (+), U16.31 (M1+)
- new net Axis_1-: M1.2 (-), U16.32 (M1-)
- new net Axis_4+: M2.1 (+), U15.31 (M1+)
- new net Axis_4-: M2.2 (-), U15.32 (M1-)
- new net Axis_5+: M3.1 (+), U15.33 (M2+)
- new net Axis_5-: M3.2 (-), U15.34 (M2-)
- new net Axis_6+: U16.33 (M2+)
- new net Axis_6-: U16.34 (M2-)
- new net CAN_GND: U18.30 (CAN_GND), U19.30 (CAN_GND), U20.30 (CAN_GND), U21.30 (CAN_GND), U22.30 (CAN_GND), U23.30 (CAN_GND)
- new net CAN_H_ARM: J7.1 (+24V), J7.2 (GND), J8.1 (+24V), J8.2 (GND)
- new net CAN_H_DRIVETRAIN: U18.28 (CAN_H), U18.29 (CAN_L), U19.28 (CAN_H), U19.29 (CAN_L), U20.28 (CAN_H), U20.29 (CAN_L), U21.28 (CAN_H), U21.29 (CAN_L), U22.28 (CAN_H), U22.29 (CAN_L), U23.28 (CAN_H), U23.29 (CAN_L)
- new net End_Effector+: M4.1 (+), U17.31 (M1+)
- new net End_Effector-: M4.2 (-), U17.32 (M1-)
- new net Ethernet to Jetson: J6.1 (Pin_1)
- new net Ubiquiti POE: J5.1 (Pin_1)
- no-connect marks 26 -> 132
Other:
- note added: "Arm Roboclaws"
- note added: "Axis 1,2,3,4,5 and End Effector"
- note added: "CAN ARM Motors"
- note added: "Comms"
- note added: "Drivetrain"
- note removed: "BILLEE Power/Logic Board"
- note removed: "Schematic Block Diagram"
- moved on the sheet: BT1, BT2, BT3, BT4, BT5, BT6, CB1, CB2, CB3, J1, J2, J3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

Commit message: meh
Connections:
- net GPIO17: no longer U17.7 (S2)
- net GPIO9: now reaches J4.32 (Pin_32)
- net GPIO9: now also U17.7 (S2)
- no-connect marks 132 -> 166
Other:
- note added: "Science"
Changed lines of the file:
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@@
 	)
 	(rectangle
+		(start 426.72 13.97)
+		(end 581.66 138.43)
+		(stroke
+			(width 0)
+			(type dash)
+		)
+		(fill
+			(type none)
+		)
+	)
+	(rectangle
 		(start 27.178 348.488)
 		(end 89.408 395.986)
@@
 		)
 	)
+	(text "Science"
+		(exclude_from_sim no)
+		(at 430.784 15.494 0)
+		(effects
+			(font
+				(size 1.27 1.27)
+			)
+		)
+	)
 	(text "To PI4B USB"
 		(exclude_from_sim no)
@@
 	)
 	(no_connect
+		(at 34.29 274.32)
+	)
+	(no_connect
+		(at 34.29 302.26)
+	)
+	(no_connect
 		(at 152.4 276.86)
 	)
@@
 	)
 	(no_connect
+		(at 34.29 292.1)
+	)
+	(no_connect
 		(at 499.11 212.09)
 	)
@@
 	)
 	(no_connect
+		(at 34.29 266.7)
+	)
+	(no_connect
 		(at 527.05 179.07)
 	)
@@
 	)
 	(no_connect
+		(at 34.29 289.56)
+	)
+	(no_connect
 		(at 152.4 284.48)
 	)
@@
 	)
 	(no_connect
+		(at 34.29 264.16)
+	)
+	(no_connect
 		(at 218.44 274.32)
 	)
 	(no_connect
+		(at 72.39 297.18)
+	)
+	(no_connect
 		(at 182.88 327.66)
 	)
@@
 	)
 	(no_connect
+		(at 72.39 264.16)
+	)
+	(no_connect
 		(at 391.16 287.02)
 	)
@@
 	)
 	(no_connect
+		(at 72.39 304.8)
+	)
+	(no_connect
 		(at 116.84 314.96)
 	)
@@
 	)
 	(no_connect
+		(at 34.29 297.18)
+	)
+	(no_connect
 		(at 182.88 325.12)
 	)
 	(no_connect
+		(at 34.29 259.08)
+	)
+	(no_connect
 		(at 78.74 201.93)
 	)
 	(no_connect
+		(at 72.39 271.78)
+	)
+	(no_connect
 		(at 116.84 312.42)
 	)
@@
 	)
 	(no_connect
+		(at 34.29 294.64)
+	)
+	(no_connect
 		(at 250.19 325.12)
 	)
 	(no_connect
+		(at 34.29 276.86)
+	)
+	(no_connect
 		(at 218.44 284.48)
 	)
@@
 	)
 	(no_connect
+		(at 72.39 287.02)
+	)
+	(no_connect
+		(at 34.29 261.62)
+	)
+	(no_connect
 		(at 386.08 361.95)
 	)
@@
 	)
 	(no_connect
+		(at 34.29 304.8)
+	)
+	(no_connect
+		(at 72.39 289.56)
+	)
+	(no_connect
+		(at 72.39 299.72)
+	)
+	(no_connect
 		(at 177.8 116.84)
 	)
@@
 	)
 	(no_connect
+		(at 34.29 299.72)
+	)
+	(no_connect
 		(at 66.04 330.2)
 	)
 	(no_connect
+		(at 34.29 281.94)
+	)
+	(no_connect
 		(at 527.05 328.93)
 	)
 	(no_connect
+		(at 72.39 284.48)
+	)
+	(no_connect
 		(at 250.19 276.86)
 	)
@@
 	)
 	(no_connect
+		(at 72.39 259.08)
+	)
+	(no_connect
 		(at 50.8 96.52)
 	)
@@
 	)
 	(no_connect
+		(at 34.29 279.4)
+	)
+	(no_connect
 		(at 218.44 279.4)
 	)
@@
 	)
 	(no_connect
+		(at 34.29 284.48)
+	)
+	(no_connect
 		(at 27.94 199.39)
 	)
@@
 	)
 	(no_connect
+		(at 72.39 292.1)
+	)
+	(no_connect
 		(at 182.88 274.32)
 	)
@@
 	)
 	(no_connect
+		(at 72.39 302.26)
+	)
+	(no_connect
 		(at 116.84 279.4)
 	)
@@
 	)
 	(no_connect
+		(at 34.29 269.24)
+	)
+	(no_connect
 		(at 116.84 287.02)
 	)
@@
 	)
 	(no_connect
+		(at 34.29 271.78)
+	)
+	(no_connect
 		(at 250.19 317.5)
 	)
@@
 	)
 	(no_connect
+		(at 72.39 269.24)
+	)
+	(no_connect
 		(at 391.16 361.95)
 	)
@@
 	)
 	(no_connect
+		(at 34.29 256.54)
+	)
+	(no_connect
 		(at 27.94 191.77)
 	)
@@
 	)
 	(no_connect
+		(at 34.29 287.02)
+	)
+	(no_connect
+		(at 72.39 279.4)
+	)
+	(no_connect
 		(at 27.94 214.63)
 	)
@@
 	)
 	(no_connect
+		(at 72.39 266.7)
+	)
+	(no_connect
 		(at 170.18 95.25)
 	)
@@
 		)
 	)
-	(global_label "GPIO17"
+	(global_label "Jetson_+5V"
 		(shape input)
-		(at 250.19 284.48 180)
+		(at 250.19 261.62 180)
 		(fields_autoplaced yes)
 		(effects
@@
 		)
 		(property "Intersheetrefs" "${INTERSHEET_REFS}"
-			(at 240.3105 284.48 0)
+			(at 236.2587 261.62 0)
 			(effects
 				(font
@@
 		)
 	)
-	(global_label "Jetson_+5V"
+	(global_label "GPIO9"
 		(shape input)
-		(at 250.19 261.62 180)
+		(at 72.39 294.64 0)
+		(fields_autoplaced yes)
+		(effects
+			(font
+				(size 1.27 1.27)
+			)
+			(justify left)
+		)
+		(property "Intersheetrefs" "${INTERSHEET_REFS}"
+			(at 81.06 294.64 0)
+			(effects
+				(font
+					(size 1.27 1.27)
+				)
+				(justify left)
+				(hide yes)
+			)
+		)
+	)
+	(global_label "GPIO9"
+		(shape input)
+		(at 250.19 284.48 180)
 		(fields_autoplaced yes)
 		(effects
@@
 		)
 		(property "Intersheetrefs" "${INTERSHEET_REFS}"
-			(at 236.2587 261.62 0)
+			(at 241.52 284.48 0)
 			(effects
 				(font
@@
 		(dnp no)
 		(property "Reference" "J7"
-			(at 237.49 393.954 0)
+			(at 228.346 393.954 0)
 			(effects
 				(font
@@
 		)
 		(property "Value" "P-20-90-PRO-121-B"
-			(at 247.65 395.986 0)
+			(at 238.506 395.986 0)
 			(effects
 				(font

Commit message: Done missing science
Parts:
- removed M2, M3, M4: Yellowjacket 5203, symbol logic_board:Yellowjacket 5203
- removed U17: RoboClaw_2x7A, symbol logic_board:RoboClaw_2x7A
- added M2, M3: FGA-32124500-G1166, symbol logic_board:FGA-32124500-G1166
- added M4: CN-PA36-38244500-G369, symbol logic_board:CN-PA36-38244500-G369
- added R7, R8, R9: 2k, symbol Device:R_US
- added U24, U25, U26: 5k (8mm Bore), symbol logic_board:NP32HS
Connections:
- net Axis_6+ is gone; now on net End_Effector+: U16.33 (M2+)
- net Axis_6- is gone; now on net End_Effector-: U16.34 (M2-)
- net Axis_4+: now also M2.1 (+)
- net Axis_4-: now also M2.2 (-)
- net Axis_5+: now also M3.1 (+)
- net Axis_5-: now also M3.2 (-)
- net End_Effector+: now also M4.1 (+)
- net End_Effector-: now also M4.2 (-)
- net at U16.27 (EN2+): now also U25.2
- net at U16.29 (EN2_5V): now also R7.1
- net at U16.30 (EN2_GND): now also U25.1
- net at U15.23 (EN1+): now also U24.2
- net at U15.25 (EN1_5V): now also R8.1
- net at U15.26 (EN1_GND): now also U24.1
- net at U15.27 (EN2+): now also U26.2
- net at U15.29 (EN2_5V): now also R9.1
- net at U15.30 (EN2_GND): now also U26.1
- new net: R7.2, U25.3
- new net: R9.2, U26.3
- new net: R8.2, U24.3
- no-connect marks 166 -> 130
Other:
- moved on the sheet: U15, U16

Commit message: updates
Connections:
- no-connect marks 130 -> 133
Other:
- moved on the sheet: J4
