File: mercury-1/mercury-1.kicad_sch (KiCad schematic)
At the start: 76 parts, among them J1 +22.2V Logic Battery Array, J2 +14.4V Drivetrain Battery Arr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, J3 +22.2V A/S Battery Array, J4 Jetson, J5 POE Injector, J6 Network Switch, J7 P-20-90-PRO-121-B, J8 P-20-90-PRO-121-B, K1 200A Relay 12V Coil, K2 200A Relay 12V Coil, K3 200A Relay 12V Coil, K4 200A Relay 12V Coil, K5 200A Relay 12V Coil, K6 200A Relay 12V Coil, K7 200A Relay 12V Coil, K8 200A Relay 12V Coil, M1 Yellowjacket 5203, M10 NEO_Brushless_Motor, M2 FGA-32124500-G1166, M3 FGA-32124500-G1166, M4 CN-PA36-38244500-G369, M5 NEO_Brushless_Motor, M6 NEO_Brushless_Motor, M7 NEO_Brushless_Motor, M8 NEO_Brushless_Motor, M9 NEO_Brushless_Motor, SW1 SW_SPDT_321, U1 UVLO Relay, U10 MAX6675 Breakout, U11 MAX6675 Breakout, U12 MAX6675 Breakout, U13 MAX6675 Breakout, U14 MAX6675 Breakout, U15 RoboClaw_2x7A, U16 RoboClaw_2x7A, U18 ODESC_V4.2, U19 ODESC_V4.2, U2 Buck Converter, U20 ODESC_V4.2, U21 ODESC_V4.2, U22 ODESC_V4.2, U23 ODESC_V4.2, U24 5k (8mm Bore), U25 5k (8mm Bore), U26 5k (8mm Bore), U3 Buck Converter, U4 UVLO Relay, U5 Logic Relay, U6 Logic Relay, U7 UVLO Relay, U8 RASPBERRY_PI_4B_4GB, U9 MAX6675 Breakout

Commit message: go to your 9am
Parts:
- R7, R8, R9: value 2k -> 7.5k
Changed lines of the file:
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@@
 			)
 		)
-		(property "Value" "2k"
+		(property "Value" "7.5k"
 			(at 265.43 289.5599 0)
 			(effects
@@
 			)
 		)
-		(property "Value" "2k"
+		(property "Value" "7.5k"
 			(at 265.43 276.8599 0)
 			(effects
@@
 			)
 		)
-		(property "Value" "2k"
+		(property "Value" "7.5k"
 			(at 199.39 289.5599 0)
 			(effects
