File: mercury-1/science.kicad_sch (KiCad schematic)
At the start: 25 parts, among them M11 Pump3, M12 Pump2, M13 Pump1, M14 Linear Actuator, M15 Stirrer, M16 Drill, M17 Drill Module 1, M18 Drill Module 2, M19 Servo 1, M20 Servo 2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

Commit message: Added EStop in code and Schematic
Parts:
- added SW2: E-Stop Drill Module 1, Button_Switch_SMD:Nidec_Copal_CAS-120A, symbol Switch:SW_Nidec_CAS-120A1
- added SW3: E-Stop Drill Module 2, Button_Switch_SMD:Nidec_Copal_CAS-120A, symbol Switch:SW_Nidec_CAS-120A1
Connections:
- net +6V: no longer U32.26 (VDD)
- net GND: now also SW2.3 (A), SW3.3 (A)
- net ardu_+5V: now reaches A1.5V1 (5V)
- net ardu_+5V: now also U32.26 (VDD)
- net e_stop_DrillM1: now reaches A1.D13
- net e_stop_DrillM1: now also SW2.2 (B)
- net e_stop_DrillM2: now reaches A1.D14 (D14/TX3)
- net e_stop_DrillM2: now also SW3.2 (B)
- no-connect marks 62 -> 90
